File: KiCad/GSM-Alarmanlage.kicad_pcb (KiCad board)
At the start: 2 copper layers, 87.5 x 79.3 mm, 23 parts, among them J1 Power, J2 Scharf / unscharf, J3 Bew. Melder, J4 Kontakte, U1 CRE1S1205SC, U2 SIM800L_7-Pin, U3 Arduino_nano

Commit message: Add files via upload
Parts:
- removed REF**: OSHW-Logo2_9.8x8mm_SilkScreen, Symbol:OSHW-Logo2_9.8x8mm_SilkScreen
- moved U2 0.07 mm to (162.3, 70.8)
- renumbered U3 to Ar1
Routing:
- net Net-(Ar1-Pad7): track 54.8 -> 57.6 mm
- net Net-(Ar1-Pad8): track 50.5 -> 51.4 mm
Other:
- board text added: "GSM Alarmmelder Rev.2 May 14. 2021 Hans-J.R. open-boat-projects.org CC BY-NC-SA"
- board text removed: "GSM Alarmmelder Rev.1 May 1. 2021 Hans-J.R. open-boat-projects.org CC BY-NC-SA"
