File: KiCad/GSM-Alarmanlage.kicad_pcb (KiCad board)
At the start: 2 copper layers, 87.5 x 79.3 mm, 22 parts, among them J1 Power, J2 Scharf / unscharf, J3 Bew. Melder, J4 Kontakte, U1 CRE1S1205SC, U2 SIM800L_7-Pin

Commit message: Add files via upload
Parts:
- R1, R2, R3: footprint Resistor_THT:R_Axial_DIN0204_L3.6mm_D1.6mm_P7.62mm_Horizontal -> Resistor_THT:R_Axial_DIN0309_L9.0mm_D3.2mm_P12.70mm_Horizontal
- moved R3 17.7 mm to (145.3, 100.6), turned to 270 degrees
- moved R2 13.1 mm to (149.3, 100.6), turned to 270 degrees
- moved R1 13.0 mm to (140.0, 113.1)
Routing:
- net Net-(D2-Pad2): track 7.95 -> 18.3 mm
- net Net-(D1-Pad2): track 8.05 -> 12.1 mm
- net GND: track 178.6 -> 181.8 mm
- net +5V: track 173.6 -> 175.0 mm
- net D7: track 75.8 -> 76.6 mm, vias 0 -> 1
- net Net-(Ar1-Pad7): track 57.6 -> 58.4 mm
