File: KiCad/GSM-Alarmanlage.sch (KiCad schematic (older format))
At the start: 22 parts, among them J1 Power, J2 Scharf / unscharf, J3 Bew. Melder, J4 Kontakte, U1 CRE1S1205SC, U2 SIM800L_7-Pin

Commit message: Add files via upload
Parts:
- R1, R2, R3: footprint Resistor_THT:R_Axial_DIN0204_L3.6mm_D1.6mm_P7.62mm_Horizontal -> Resistor_THT:R_Axial_DIN0309_L9.0mm_D3.2mm_P12.70mm_Horizontal
Changed lines of the file:
@@
 F 0 "R3" H 7709 4696 50  0000 L CNN
 F 1 "330" H 7709 4605 50  0000 L CNN
-F 2 "Resistor_THT:R_Axial_DIN0204_L3.6mm_D1.6mm_P7.62mm_Horizontal" H 7650 4650 50  0001 C CNN
+F 2 "Resistor_THT:R_Axial_DIN0309_L9.0mm_D3.2mm_P12.70mm_Horizontal" H 7650 4650 50  0001 C CNN
 F 3 "~" H 7650 4650 50  0001 C CNN
 	1    7650 4650
@@
 F 0 "R2" H 7459 4896 50  0000 L CNN
 F 1 "330" H 7459 4805 50  0000 L CNN
-F 2 "Resistor_THT:R_Axial_DIN0204_L3.6mm_D1.6mm_P7.62mm_Horizontal" H 7400 4850 50  0001 C CNN
+F 2 "Resistor_THT:R_Axial_DIN0309_L9.0mm_D3.2mm_P12.70mm_Horizontal" H 7400 4850 50  0001 C CNN
 F 3 "~" H 7400 4850 50  0001 C CNN
 	1    7400 4850
@@
 F 0 "R1" H 3059 2896 50  0000 L CNN
 F 1 "10k" H 3059 2805 50  0000 L CNN
-F 2 "Resistor_THT:R_Axial_DIN0204_L3.6mm_D1.6mm_P7.62mm_Horizontal" H 3000 2850 50  0001 C CNN
+F 2 "Resistor_THT:R_Axial_DIN0309_L9.0mm_D3.2mm_P12.70mm_Horizontal" H 3000 2850 50  0001 C CNN
 F 3 "~" H 3000 2850 50  0001 C CNN
 	1    3000 2850
